File: L298.kicad_sch (KiCad schematic)
At the start: 18 parts, among them U2 L298HN, U3 INA226, U4 INA226, U6 INA226, U7 INA226

Commit message: Added Footprint
Parts:
- C24: footprint (none) -> Capacitor_THT:CP_Radial_D5.0mm_P2.00mm
- R5, R6, R8, R9: footprint (none) -> Resistor_SMD:R_2512_6332Metric_Pad1.40x3.35mm_HandSolder
Changed lines of the file:
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@@
 			)
 		)
-		(property "Footprint" ""
+		(property "Footprint" "Resistor_SMD:R_2512_6332Metric_Pad1.40x3.35mm_HandSolder"
 			(at 98.552 120.65 90)
 			(effects
@@
 			)
 		)
-		(property "Footprint" ""
+		(property "Footprint" "Capacitor_THT:CP_Radial_D5.0mm_P2.00mm"
 			(at 187.6552 38.1 0)
 			(effects
@@
 			)
 		)
-		(property "Footprint" ""
+		(property "Footprint" "Resistor_SMD:R_2512_6332Metric_Pad1.40x3.35mm_HandSolder"
 			(at 154.432 119.38 90)
 			(effects
@@
 			)
 		)
-		(property "Footprint" ""
+		(property "Footprint" "Resistor_SMD:R_2512_6332Metric_Pad1.40x3.35mm_HandSolder"
 			(at 41.402 124.46 90)
 			(effects
@@
 			)
 		)
-		(property "Footprint" ""
+		(property "Footprint" "Resistor_SMD:R_2512_6332Metric_Pad1.40x3.35mm_HandSolder"
 			(at 209.042 118.11 90)
 			(effects

Commit message: FInal Changes in Schgematic
Parts:
- removed R5, R6, R8, R9: 50m, Resistor_SMD:R_2512_6332Metric_Pad1.40x3.35mm_HandSolder, symbol Device:R
- removed U3, U4, U6, U7: INA226, Package_SO:VSSOP-10_3x3mm_P0.5mm, symbol Sensor_Energy:INA226
Connections:
- net OUT1 is gone; now on net MOTOR1+: D1.2 (A), D2.1 (K), U2.2 (OUT1)
- net OUT2 is gone; now on net MOTOR1-: D3.1 (K), D6.2 (A), U2.3 (OUT2)
- net OUT3 is gone; now on net MOTOR2+: D4.1 (K), D7.2 (A), U2.13 (OUT3)
- net OUT4 is gone; now on net MOTOR2-: D5.1 (K), D8.2 (A), U2.14 (OUT4)
- net +15V renamed +15
- net +5V renamed +5
- no-connect marks 4 -> 0
Other:
- moved on the sheet: C24, D1, D2, D3, D4, D5, D6, D7, D8, U2

Commit message: Made Changes to Layout and USB C
Parts:
- U2: footprint Package_TO_SOT_THT:TO-220-15_P2.54x2.54mm_StaggerOdd_Lead5.84mm_TabDown -> Package_TO_SOT_THT:TO-220-15_P2.54x5.08mm_StaggerEven_Lead4.58mm_Vertical
Changed lines of the file:
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@@
 			)
 		)
-		(property "Footprint" "Package_TO_SOT_THT:TO-220-15_P2.54x2.54mm_StaggerOdd_Lead5.84mm_TabDown"
+		(property "Footprint" "Package_TO_SOT_THT:TO-220-15_P2.54x5.08mm_StaggerEven_Lead4.58mm_Vertical"
 			(at 105.41 105.41 0)
 			(effects
