File: MNAPcb.kicad_sch (KiCad schematic)
At the start: 14 parts, among them J1 Conn_01x03_Pin, J2 DA15_Socket, J3 USB_C_Receptacle_USB2.0_16P, J5 Conn_01x02, J7 Conn_01x02, J8 Conn_01x04_Pin, J9 Conn_01x02

Commit message: Solved all the Erros
Parts:
- J3: footprint Connector_USB:USB_C_Receptacle_G-Switch_GT-USB-7010ASV -> Connector_USB:USB_C_Receptacle_Palconn_UTC16-G
Changed lines of the file:
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@@
 			)
 		)
-		(property "Footprint" "Connector_USB:USB_C_Receptacle_G-Switch_GT-USB-7010ASV"
+		(property "Footprint" "Connector_USB:USB_C_Receptacle_Palconn_UTC16-G"
 			(at 219.71 120.65 0)
 			(effects
